File: Sirena/KiCad/Sirena.sch (KiCad schematic (older format))
At the start: 12 parts

Commit message: aggiornato schema Sirena eliminando tutti i circuiti aggiuntivi
Parts:
- removed Dev?: ALIMENTATORE, ~, symbol ALIMENTATORE
- removed K?: RELAY_1RT, ~, symbol RELAY_1RT
- removed MM? (x2): MAMMUTH02, ~, symbol MAMMUTH02
- removed MM?: MAMMUTH03, ~, symbol MAMMUTH03
- removed MM?: MAMMUTH10, ~, symbol MAMMUTH10
- removed MM?: MAMMUTH01, ~, symbol MAMMUTH01
- removed MM?: MAMMUTH12, ~, symbol MAMMUTH12
- removed MM?: MAMMUTH_07, ~, symbol MAMMUTH_07
- removed SW?: PwrSwitch, ~, symbol SINGLE_SWITCH
- added MM1, MM2: MAMMUTH_06, ~, symbol MAMMUTH_06
- gave numbers to parts that had none: 2
Connections:
- net labels removed: +12Vcc - OUT, +12Vcc Internal, -Batt, 12V-Switch
- wire segments 80 -> 38
Other:
- note removed: "Black"
- note removed: "Blue"
- note removed: "Orange"
- note removed: "Red"
