File: Lampada/KiCAD/Lampada.kicad_pcb (KiCad board)
At the start: 2 copper layers, 6 parts, among them IC1 4N35, IC2 4N35, SW1 default

Commit message: 2015-02-16 07:38 - commit with no comment
Parts:
- removed MM1: MAMMUTH_07, LnSIP-07
- removed R2: 680, LnRes-500
- removed SW1: default, LnSIP-02
- added DL1: LED, LnLED-5MM, F.Cu at (96.5, 73.7)
- IC1, IC2: footprint LnDIP-06_300 -> DIP-6__300
- R1: value 4K7 -> 2K7
- moved IC2 103.4 mm to (86.4, 73.7), turned to 270 degrees
- moved R1 94.8 mm to (95.2, 64.8)
- moved IC1 83.2 mm to (101.6, 55.9), turned to 90 degrees
Connections:
- IC1 pad 1: N-0000022 -> N-0000013
- IC2 pad 1: /c2 -> (no net)
- IC2 pad 2: GNDA -> (no net)
- IC2 pad 4: (no net) -> GNDA
- IC2 pad 5: (no net) -> /c2
- R1 pad 1: N-0000022 -> N-0000024
