File: Lampada/KiCAD/Lampada.sch (KiCad schematic (older format))
At the start: 11 parts, among them IC1 4N35, IC2 4N35, K1 RELAY_1RT, Q1 NPN, SW1 default

Commit message: 2015-02-16 07:38 - commit with no comment
Parts:
- added D2: DIODE, ~, symbol DIODE
- added DL1, DL2, DL3: LED, ~, symbol LED
- added IC3, IC4: 4N35, DIP6, symbol 4N35
- added J1: SIP_04, ~, symbol SIP_04
- added K2: RELAY_1RT, ~, symbol RELAY_1RT
- added Q2: NPN, ~, symbol NPN
- added R4: 1k, ~, symbol RESISTOR
- added R5: 2K7, ~, symbol RESISTOR
- added R6: 10K, ~, symbol RESISTOR
- added SW2, SW4: Manual ON, ~, symbol SINGLE_SWITCH
- added SW3: default, ~, symbol SINGLE_SWITCH
- R1: value 4K7 -> 2K7
Connections:
- net labels added: +12V, LampON
- net labels removed: +5V
- wire segments 62 -> 107
- no-connect marks 6 -> 7
Other:
- moved on the sheet: D1, K1, Q1, R1, R2, R3
